File: VGC-0_rp_1v0/VGC-0_rp_1v0.kicad_sch (KiCad schematic)
At the start: 85 parts, among them J1 USB-TYPE-C-017, J2 BATTERY, J4 SM03B-SRSS-TB, SW1 SW_Push, SW2 SW_Push, SW3 SW_Push, SW4 SW_Push, U1 RP2350_60QFN, U2 SPX3819M5-L-3-3/TR, U3 W25Q128JVS, U4 ESP8684-MINI-1, U5 APS1604M-3SQR-ZR, U6 SPX3819M5-L-3-3/TR, U7 BQ24073RGTR, Y1 ABM8-272-T3

Commit message: power sys update 0
Parts:
- removed U2, U6: SPX3819M5-L-3-3/TR, Package_TO_SOT_SMD:SOT-23-5, symbol our-parts:SPX3819M5-L-3-3/TR
- added C30: 20u, symbol Device:C
- added C31: 100n, symbol Device:C
- added C32: 100uF, Capacitor_SMD:C_0402_1005Metric, symbol Device:C
- added J3: SMD pads for 3.3V, our-parts:SMD-solder-pad-2x, symbol our-parts:2PIN
- added L2: 2.2uH, our-parts:SMD-inductor-4mm9_4mm9, symbol Device:L
- added R27, R29: 1MR, Resistor_SMD:R_0402_1005Metric, symbol Device:R
- added R28: 120kR, Resistor_SMD:R_0603_1608Metric, symbol Device:R
- added R30: 200kR, Resistor_SMD:R_0402_1005Metric, symbol Device:R
- added R31, R33: 200R, Resistor_SMD:R_0402_1005Metric, symbol Device:R
- added R32, R34: 1k, Resistor_SMD:R_0402_1005Metric, symbol Device:R
- added U2: RT6154A, Package_DFN_QFN:DFN-14-1EP_3x4mm_P0.5mm_EP1.7x3.3mm, symbol our-parts:RT6154A
- J2: value BATTERY -> THT pins for BATTERY
- JP1: footprint (none) -> Jumper:SolderJumper-2_P1.3mm_Open_RoundedPad1.0x1.5mm
Connections:
- net +3V3: now also C32.1, J3.1 (□), R27.1, R29.1, U2.4 (Vout), U2.5 (Vout)
- net GND: now also C30.1, C31.1, C32.2, J3.2 (○), R30.2, R32.2, R34.2, U2. (P-GND), U2.2 (GND)
- net VCC: now also C30.2, U2.10 (Vin), U2.11 (Vin), U2.12 (EN)
- net at U7.12 (ILIM): now also R31.1
- net at U7.16 (ISET): now also R33.1
- new net: R28.2, R30.1, U2.3 (FB)
- new net: R33.2, R34.1
- new net: C31.2, U2.1 (VinA)
- new net: R27.2, R28.1
- new net: R29.2, U2.14 (PGOOD)
- new net: L2.2, U2.6 (LX2), U2.7 (LX2)
- new net: L2.1, U2.8 (LX1), U2.9 (LX1)
- new net: R31.2, R32.1
- no-connect marks 17 -> 16
Other:
- note added: "R1 = 1.12MR R2 = 200kR => Vout = 3.3V R1 = R2(Vout/0.5V -1)"
- note added: "R27 + R28 = 1.12MR"
- moved on the sheet: C1, C5, D2, D3, J1, J2, JP1, R22, R23, R24, R25, R26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
