File: VGC-0_rp_1v0/VGC-0_rp_1v0.kicad_sch (KiCad schematic)
At the start: 99 parts, among them J1 USB-TYPE-C-017, J2 THT pins for BATTERY, J3 SMD pads for 3.3V, J4 SM03B-SRSS-TB, SW1 SW_Push, SW2 SW_Push, SW3 SW_Push, SW4 SW_Push, U1 RP2350_60QFN, U2 RT6154A, U3 W25Q128JVS, U4 ESP8684-MINI-1, U5 APS1604M-3SQR-ZR, U7 BQ24073RGTR, Y1 ABM8-272-T3

Commit message: update rev.2.1
Parts:
- removed H2: MountingHole-M3, MountingHole:MountingHole_3mm, symbol Mechanical:MountingHole
- added C34: 100n, Capacitor_SMD:C_0402_1005Metric, symbol Device:C
- added C35: 10u, Capacitor_SMD:C_0805_2012Metric, symbol Device:C
- BTN5, BTN6: footprint our-parts:8x8-tht-button -> our-parts:THT-button_2pin
Connections:
- net +3V3: now also C34.1, C35.1
- net GND: now also U2.15 (P-GND), C34.2, C35.2; no longer U2. (P-GND)
Other:
- moved on the sheet: C1, C30, C31, C32, C33, C5, D2, D3, J1, J2, J3, JP1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

Commit message: update rev.2.2
Parts:
- added C36: 2.2u, Capacitor_SMD:C_0402_1005Metric, symbol Device:C
- C31: footprint (none) -> Capacitor_SMD:C_0402_1005Metric
- J1: footprint (none) -> our-parts:USB-TYPE-C-SMD_C9900008089
Connections:
- net BTN_START: now also C36.1
- net GND: now also C36.2
Other:
- note added: "TO DO: - add ID to 100nF caps"
- note removed: "TO DO: - add ID to 100nF caps - add footprint to J1"
- moved on the sheet: BTN1, BTN2, BTN3, BTN4, BTN5, BTN6, C19, C20, C21, C22, C23, C24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

Commit message: update rev.2.3
Connections:
- net +BATT: now also U7.2,3 (BATT); no longer U7.2 (BATT)
Changed lines of the file:
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@@
 			)
 		)
-		(pin "2"
+		(pin "2,3"
 		)
 		(pin "4"

Commit message: update rev.2.4
Parts:
- added J6: audio-out, our-parts:2.54mm-2PIN, symbol our-parts:2PIN
Connections:
- net +BATT: now also U7.2 (BATT), U7.3 (BATT); no longer U7.2,3 (BATT)
- net Audio: now also J6.1 (□)
- net GND: now also U7.8 (VSS), J6.2 (○)
- net VCC: now also U7.11 (OUT)

Commit message: update rev.2.51
Changed lines of the file:
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@@
 	(wire
 		(pts
-			(xy 48.26 358.14) (xy 45.72 358.14)
+			(xy 48.26 358.14) (xy 46.99 358.14)
 		)
 		(stroke
@@
 	(wire
 		(pts
-			(xy 45.72 358.14) (xy 45.72 361.95)
+			(xy 46.99 358.14) (xy 46.99 369.57)
 		)
 		(stroke
@@
 	(symbol
 		(lib_id "power:GND")
-		(at 45.72 361.95 0)
+		(at 46.99 369.57 0)
 		(unit 1)
 		(exclude_from_sim no)
@@
 		(dnp no)
 		(property "Reference" "#PWR015"
-			(at 45.72 368.3 0)
+			(at 46.99 375.92 0)
 			(effects
 				(font
@@
 		)
 		(property "Value" "GND"
-			(at 41.91 363.22 0)
+			(at 43.18 370.84 0)
 			(effects
 				(font
@@
 		)
 		(property "Footprint" ""
-			(at 45.72 361.95 0)
+			(at 46.99 369.57 0)
 			(effects
 				(font
@@
 		)
 		(property "Datasheet" ""
-			(at 45.72 361.95 0)
+			(at 46.99 369.57 0)
 			(effects
 				(font
@@
 		)
 		(property "Description" ""
-			(at 45.72 361.95 0)
+			(at 46.99 369.57 0)
 			(effects
 				(font
