File: VGC-0_rp_1v0/_autosave-VGC-0_rp_1v0.kicad_sch (KiCad schematic)
At the start: 99 parts, among them J1 USB-TYPE-C-017, J2 THT pins for BATTERY, J3 SMD pads for 3.3V, J4 SM03B-SRSS-TB, SW1 SW_Push, SW2 SW_Push, SW3 SW_Push, SW4 SW_Push, U1 RP2350_60QFN, U2 RT6154A, U3 W25Q128JVS, U4 ESP8684-MINI-1, U5 APS1604M-3SQR-ZR, U7 BQ24073RGTR, Y1 ABM8-272-T3

Commit message: update rev.2
Parts:
- C31: footprint (none) -> Capacitor_SMD:C_0402_1005Metric
Connections:
- net GND: now also U2.15 (P-GND); no longer U2. (P-GND)
Changed lines of the file:
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@@
 		(title "VGC-0-rpi")
 		(date "2025-08-08")
-		(rev "REV2")
+		(rev "2")
 		(company "Chili Chip")
 		(comment 1 "This is a prototype")
@@
 	(text "TO DO: \n- add ID to 100nF caps\n- add footprint to J1"
 		(exclude_from_sim no)
-		(at 474.726 378.968 0)
+		(at 474.98 380.238 0)
 		(effects
 			(font
@@
 	)
 	(symbol
-		(lib_id "Device:C")
-		(at 54.61 186.69 180)
-		(unit 1)
-		(exclude_from_sim no)
-		(in_bom yes)
-		(on_board yes)
-		(dnp no)
-		(property "Reference" "C31"
-			(at 61.468 188.214 0)
-			(effects
-				(font
-					(size 1.27 1.27)
-				)
-				(justify left)
-			)
-		)
-		(property "Value" "100n"
-			(at 62.484 185.928 0)
-			(effects
-				(font
-					(size 1.27 1.27)
-				)
-				(justify left)
-			)
-		)
-		(property "Footprint" ""
-			(at 53.6448 182.88 0)
-			(effects
-				(font
-					(size 1.27 1.27)
-				)
-				(hide yes)
-			)
-		)
-		(property "Datasheet" "~"
-			(at 54.61 186.69 0)
-			(effects
-				(font
-					(size 1.27 1.27)
-				)
-				(hide yes)
-			)
-		)
-		(property "Description" ""
-			(at 54.61 186.69 0)
-			(effects
-				(font
-					(size 1.27 1.27)
-				)
-				(hide yes)
-			)
-		)
-		(pin "1"
-		)
-		(pin "2"
-		)
-		(instances
-			(project "VGC-0_rp_1v0"
-				(path "/94683f5c-9cd9-448e-be96-9792537b5cb8"
-					(reference "C31")
-					(unit 1)
-				)
-			)
-		)
-	)
-	(symbol
 		(lib_id "Device:R")
 		(at 532.13 135.89 0)
@@
 	)
 	(symbol
+		(lib_id "Device:C")
+		(at 54.61 186.69 180)
+		(unit 1)
+		(exclude_from_sim no)
+		(in_bom yes)
+		(on_board yes)
+		(dnp no)
+		(property "Reference" "C31"
+			(at 51.689 187.8584 0)
+			(effects
+				(font
+					(size 1.27 1.27)
+				)
+				(justify left)
+			)
+		)
+		(property "Value" "100n"
+			(at 51.689 185.547 0)
+			(effects
+				(font
+					(size 1.27 1.27)
+				)
+				(justify left)
+			)
+		)
+		(property "Footprint" "Capacitor_SMD:C_0402_1005Metric"
+			(at 53.6448 182.88 0)
+			(effects
+				(font
+					(size 1.27 1.27)
+				)
+				(hide yes)
+			)
+		)
+		(property "Datasheet" "~"
+			(at 54.61 186.69 0)
+			(effects
+				(font
+					(size 1.27 1.27)
+				)
+				(hide yes)
+			)
+		)
+		(property "Description" ""
+			(at 54.61 186.69 0)
+			(effects
+				(font
+					(size 1.27 1.27)
+				)
+				(hide yes)
+			)
+		)
+		(pin "1"
+		)
+		(pin "2"
+		)
+		(instances
+			(project "VGC-0_rp_1v0"
+				(path "/94683f5c-9cd9-448e-be96-9792537b5cb8"
+					(reference "C31")
+					(unit 1)
+				)
+			)
+		)
+	)
+	(symbol
 		(lib_id "power:GND")
 		(at 41.91 190.5 0)
@@
 		(pin "9"
 		)
-		(pin ""
+		(pin "15"
 		)
 		(pin "12"
