File: VGC-0_rp_1v0/VGC-0_rp_1v0.kicad_pcb (KiCad board)
At the start: 2 copper layers, 52 x 51 mm, 43 parts, among them J1 USB_B_Micro, J2 Conn_02x18_Odd_Even, J3 Conn_02x18_Odd_Even, J4 SM03B-SRSS-TB, SW1 SW_Push, SW2 SW_Push, U1 RP2350_60QFN, U2 NCP1117-3.3_SOT223, U3 W25Q128JVS, Y1 ABM8-272-T3

Commit message: update rev.2
Parts:
- removed H3, H4: MountingHole, MountingHole:MountingHole_2.7mm_M2.5
- removed J1: USB_B_Micro, Connector_USB:USB_Micro-B_Amphenol_10103594-0001LF_Horizontal
- added BTN1: ~, our-parts:8x8-tht-button, F.Cu at (169.0, 102.0)
- added BTN2: ~, our-parts:8x8-tht-button, F.Cu at (158.0, 109.8)
- added BTN3: ~, our-parts:8x8-tht-button, F.Cu at (180.0, 109.8)
- added BTN4: ~, our-parts:8x8-tht-button, F.Cu at (169.0, 117.5)
- added BTN5: ~, our-parts:8x8-tht-button, F.Cu at (71.7, 50.2)
- added BTN6: ~, our-parts:8x8-tht-button, F.Cu at (71.7, 58.8)
- added C20: 2.2u, Capacitor_SMD:C_0402_1005Metric, F.Cu at (84.9, 66.7)
- added C21: 2.2u, Capacitor_SMD:C_0402_1005Metric, F.Cu at (178.5, 102.0)
- added C22: 2.2u, Capacitor_SMD:C_0402_1005Metric, F.Cu at (84.9, 68.7)
- added C23: 2.2u, Capacitor_SMD:C_0402_1005Metric, F.Cu at (84.9, 70.7)
- added C24: 2.2u, Capacitor_SMD:C_0402_1005Metric, F.Cu at (84.9, 72.6)
- added C25: 2.2u, Capacitor_SMD:C_0402_1005Metric, F.Cu at (87.8, 62.8)
- added C26: 2.2u, Capacitor_SMD:C_0402_1005Metric, F.Cu at (87.8, 64.7)
- added C27: 100n, Capacitor_SMD:C_0402_1005Metric, F.Cu at (87.8, 66.7)
- added C28: 100n, Capacitor_SMD:C_0402_1005Metric, F.Cu at (87.8, 68.7)
- added C29: 2.2u, Capacitor_SMD:C_0402_1005Metric, F.Cu at (87.8, 70.7)
- added C30: 10u, Capacitor_SMD:C_0805_2012Metric, F.Cu at (95.4, 69.3)
- added C31: 100n, Capacitor_SMD:C_0402_1005Metric, F.Cu at (94.0, 42.5)
- added C32: 100uF, Capacitor_SMD:C_1206_3216Metric, F.Cu at (96.0, 75.5)
- added C33: 10u, Capacitor_SMD:C_0805_2012Metric, F.Cu at (95.4, 72.3)
- added D1: LED, Diode_SMD:D_0603_1608Metric, F.Cu at (91.4, 53.8)
- added D2: LED, Diode_SMD:D_0603_1608Metric, F.Cu at (91.4, 56.4)
- added D3: LED, Diode_SMD:D_0603_1608Metric, F.Cu at (91.4, 58.9)
- added E1: ~, our-parts:mouse-encoder, F.Cu at (186.0, 57.5)
- added J5: ~, our-parts:2.54mm-10PIN, F.Cu at (182.1, 131.0)
- added JP1: BYPASS_BATTERY, Jumper:SolderJumper-2_P1.3mm_Open_RoundedPad1.0x1.5mm, B.Cu at (134.2, 117.5)
- added L2: 2.2uH, our-parts:SMD-inductor-4mm9_4mm9, F.Cu at (93.7, 49.6)
- added LCD1: ~, our-parts:THT-SPI-LCD, F.Cu at (169.0, 92.0)
- added R11: 10k, Resistor_SMD:R_0402_1005Metric, F.Cu at (82.1, 48.9)
- added R12: 10k, Resistor_SMD:R_0402_1005Metric, F.Cu at (82.1, 50.8)
- added R13: 10k, Resistor_SMD:R_0402_1005Metric, F.Cu at (82.1, 52.8)
- added R14: 10k, Resistor_SMD:R_0402_1005Metric, F.Cu at (82.1, 54.8)
- added R15: 10k, Resistor_SMD:R_0402_1005Metric, F.Cu at (82.1, 56.8)
- added R16: 12k, Resistor_SMD:R_0402_1005Metric, F.Cu at (82.1, 58.8)
- added R17: 12k, Resistor_SMD:R_0402_1005Metric, F.Cu at (82.1, 60.8)
- added R18: 2.2k, Resistor_SMD:R_0402_1005Metric, F.Cu at (85.0, 46.9)
- added R19: 10k, Resistor_SMD:R_0402_1005Metric, F.Cu at (85.0, 48.9)
- added R20: 10k, Resistor_SMD:R_0402_1005Metric, F.Cu at (85.0, 50.8)
- added R21: 10k, Resistor_SMD:R_0402_1005Metric, F.Cu at (85.0, 52.8)
- added R22: 5.1k, Resistor_SMD:R_0402_1005Metric, F.Cu at (85.0, 54.8)
- added R23: 5.1k, Resistor_SMD:R_0402_1005Metric, F.Cu at (85.0, 56.8)
- added R24: 10k, Resistor_SMD:R_0402_1005Metric, F.Cu at (85.0, 58.8)
- added R25: 5.1k, Resistor_SMD:R_0402_1005Metric, F.Cu at (85.0, 60.8)
- added R26: 5.1k, Resistor_SMD:R_0402_1005Metric, F.Cu at (87.9, 46.9)
- added R27: 1MR, Resistor_SMD:R_0402_1005Metric, F.Cu at (87.9, 48.9)
- added R28: 120kR, Resistor_SMD:R_0603_1608Metric, F.Cu at (91.2, 73.1)
- added R29: 1MR, Resistor_SMD:R_0402_1005Metric, F.Cu at (87.9, 50.8)
- added R3: 10k, Resistor_SMD:R_0402_1005Metric, F.Cu at (79.2, 50.8)
- added R30: 200kR, Resistor_SMD:R_0402_1005Metric, F.Cu at (87.9, 52.8)
- added R31: 200R, Resistor_SMD:R_0402_1005Metric, F.Cu at (87.9, 54.8)
- added R32: 1k, Resistor_SMD:R_0402_1005Metric, F.Cu at (87.9, 56.8)
- added R33: 200R, Resistor_SMD:R_0402_1005Metric, F.Cu at (87.9, 58.8)
- added R34: 1k, Resistor_SMD:R_0402_1005Metric, F.Cu at (87.9, 60.8)
- added SW3: SW_Push, Button_Switch_SMD:SW_SPST_TL3342, F.Cu at (149.5, 90.5)
- added SW4: SW_Push, Button_Switch_SMD:SW_SPST_TL3342, F.Cu at (188.5, 90.0)
- added U4: ESP8684-MINI-1, our-parts:ESP8684-MINI-1, B.Cu at (168.5, 55.7)
- added U5: APS1604M-3SQR-ZR, our-parts:USON-8, F.Cu at (96.1, 59.8)
- added U7: BQ24073RGTR, Package_DFN_QFN:QFN-16-1EP_3x3mm_P0.5mm_EP1.7x1.7mm, F.Cu at (80.4, 76.3)
- C19: value 10u -> 2.2u; footprint Capacitor_SMD:C_0805_2012Metric -> Capacitor_SMD:C_0402_1005Metric
- C6, C7: footprint RP2350_60QFN_minimal:C_0402_1005Metric_small_pads -> Capacitor_SMD:C_0603_1608Metric
- C9: footprint Capacitor_SMD:C_0402_1005Metric -> Capacitor_SMD:C_0603_1608Metric
- H1, H2: value MountingHole -> MountingHole-M3; footprint MountingHole:MountingHole_2.7mm_M2.5 -> MountingHole:MountingHole_3mm
- J2: value Conn_02x18_Odd_Even -> THT pins for BATTERY; footprint Connector_PinHeader_2.54mm:PinHeader_2x18_P2.54mm_Vertical -> our-parts:2.54mm-2PIN
- J3: value Conn_02x18_Odd_Even -> SMD pads for 3.3V; footprint Connector_PinHeader_2.54mm:PinHeader_2x18_P2.54mm_Vertical -> our-parts:SMD-solder-pad-2x; moved to B.Cu
- J4, U1: moved to B.Cu
- R1: value DNF -> 10k
- R5: footprint Resistor_SMD:R_0402_1005Metric -> Resistor_SMD:R_0603_1608Metric
- R9: value DNF -> 0
- SW1, SW2: footprint Button_Switch_SMD:SW_Push_1P1T_NO_Vertical_Wuerth_434133025816 -> Button_Switch_SMD:SW_SPST_TL3342
- U2: value NCP1117-3.3_SOT223 -> RT6154A; footprint Package_TO_SOT_SMD:SOT-223-3_TabPin2 -> Package_DFN_QFN:DFN-14-1EP_3x4mm_P0.5mm_EP1.7x3.3mm
- moved J2 96.1 mm to (153.3, 131.0)
- moved H1 90.4 mm to (169.0, 110.0)
- moved J4 89.1 mm to (188.5, 75.5), turned to -90 degrees
- moved U1 73.0 mm to (168.7, 75.5), turned to 180 degrees
- moved R4 66.9 mm to (79.2, 52.8), turned to 0 degrees
- moved R2 61.5 mm to (79.2, 48.9), turned to 0 degrees
- moved J3 61.5 mm to (146.9, 130.0)
- moved SW1 60.6 mm to (149.5, 58.5), turned to 90 degrees
- moved SW2 54.2 mm to (149.5, 68.5), turned to -90 degrees
- moved C3 48.3 mm to (79.1, 64.7), turned to 0 degrees
- moved C4 47.9 mm to (79.1, 66.7)
- moved C18 45.3 mm to (84.9, 62.8), turned to 0 degrees
- moved H2 44.6 mm to (69.4, 73.6)
- moved C10 42.2 mm to (79.1, 70.7), turned to 0 degrees
- moved C14 42.0 mm to (82.0, 66.7)
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Connections:
- C19 pad 1: +3V3 -> ENC-A
- C5 pad 1: +3V3 -> +BATT
- J2 pad 1: GND -> +BATT
- J2 pad 2: +3V3 -> GND
- J3 pad 1: /GPIO29_ADC3 -> +3V3
- R9 pad 2: /FLASH_SS -> Net-(U5-CE)
- U1 pad 10: /GPIO7 -> Audio
- U1 pad 16: /GPIO12 -> PUPPY_RX
- U1 pad 17: /GPIO13 -> PUPPY_TX
- U1 pad 18: /GPIO14 -> PUPPY_WIFI_EN
- U1 pad 19: /GPIO15 -> PUPPY_WIFI_BOOT
- U1 pad 27: /GPIO16 -> BTN_START
- U1 pad 28: /GPIO17 -> BTN_ESC
- U1 pad 29: /GPIO18 -> ENC-A
- U1 pad 3: /GPIO1 -> LCD_PUPPY_SELECT
- U1 pad 31: /GPIO19 -> ENC-B
- U1 pad 32: /GPIO20 -> BTN1
- U1 pad 33: /GPIO21 -> BTN2
- U1 pad 34: /GPIO22 -> BTN3
- U1 pad 35: /GPIO23 -> BTN4
- U1 pad 36: /GPIO24 -> BTN5
- U1 pad 37: /GPIO25 -> BTN6
- U1 pad 4: /GPIO2 -> LCD_SCK
- U1 pad 40: /GPIO26_ADC0 -> +BATT
- U1 pad 5: /GPIO3 -> LCD_SDA
- U1 pad 7: /GPIO4 -> LCD_LED
- U1 pad 8: /GPIO5 -> LCD_A0
- U1 pad 9: /GPIO6 -> LCD_RESET
- U2 pad 1: GND -> Net-(U2-VinA)
- U2 pad 2: +3V3 -> GND
- U2 pad 3: VBUS -> Net-(U2-FB)
Routing:
- net /GPIO0: track 39.0 -> 0.00 mm, vias 2 -> 0
- net +3V3: track 37.6 -> 0.00 mm, vias 2 -> 0
- net GND: track 37.5 -> 0.00 mm, vias 27 -> 0
- net /GPIO29_ADC3: track 33.6 -> 0.00 mm
- net /GPIO28_ADC2: track 31.9 -> 0.00 mm
- net /GPIO27_ADC1: track 30.3 -> 0.00 mm
- net /GPIO1: track 29.8 -> 0.00 mm
- net /GPIO26_ADC0: track 28.6 -> 0.00 mm
- net /GPIO2: track 28.2 -> 0.00 mm
- net /SWCLK: track 27.8 -> 0.00 mm
- net /GPIO25: track 27.7 -> 0.00 mm
- net /GPIO3: track 26.5 -> 0.00 mm
- net /GPIO24: track 26.1 -> 0.00 mm
- net /SWD: track 25.4 -> 0.00 mm
- net /GPIO15: track 25.2 -> 0.00 mm
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- removed copper zone on F.Cu, net +1V1
- removed copper zone on F.Cu, net +3V3
- removed copper zone on F.Cu, net /VREG_LX
- removed copper zone on B.Cu, net GND
- removed copper zone on F.Cu, net GND
- removed copper zone on F.Cu, net VBUS
Other:
- board outline removed
- board text removed: "3V3"
- board text removed: "ADC 26-29"
- board text removed: "BOOTSEL"
- board text removed: "DEBUG"
- board text removed: "GND"
- board text removed: "GP0"
- board text removed: "GP1"
- board text removed: "GP10"
- board text removed: "GP11"
- board text removed: "GP12"
- board text removed: "GP13"
- board text removed: "GP14"
- board text removed: "GP15"
- board text removed: "GP16"
- board text removed: "GP17"
- board text removed: "GP18"
- board text removed: "GP19"
- board text removed: "GP2"
- board text removed: "GP20"
- board text removed: "GP21"
- board text removed: "GP22"
- board text removed: "GP23"
- board text removed: "GP24"
- board text removed: "GP25"
- board text removed: "GP26"
- board text removed: "GP27"
- board text removed: "GP28"
- board text removed: "GP29"
- board text removed: "GP3"
- board text removed: "GP4"
- board text removed: "GP5"
- board text removed: "GP6"
- board text removed: "GP7"
- board text removed: "GP8"
- board text removed: "GP9"
- board text removed: "Minimal Design Example REV3"
- board text removed: "Outer Row GND"
- board text removed: "RUN"
- board text removed: "Raspberry Pi RP2350A QFN-60"
- board text removed: "SWCLK"
- board text removed: "SWD"

Commit message: update rev.2.1
Parts:
- removed H2: MountingHole-M3, MountingHole:MountingHole_3mm
- added C34: 100n, Capacitor_SMD:C_0402_1005Metric, B.Cu at (171.7, 56.6)
- added C35: 10u, Capacitor_SMD:C_0805_2012Metric, B.Cu at (172.2, 54.5)
- BTN5, BTN6: footprint our-parts:8x8-tht-button -> our-parts:THT-button_2pin
- C1, C2, C21, C27, C28, C3, C30, C31, C32, C33, C4, C5, D1, L1, L2, R1, R10, R15, R18, R19, R2, R24, R27, R28, R29, R30, R31, R32, R33, R34, R9, U2, U3, U5, U7, Y1: moved to B.Cu
- JP1: moved to F.Cu
- moved R27 127.2 mm to (191.2, 123.0), turned to 180 degrees
- moved BTN5 123.7 mm to (180.0, 109.8), turned to 90 degrees
- moved L2 120.0 mm to (182.8, 130.0)
- moved R30 119.9 mm to (186.1, 121.6), turned to 90 degrees
- moved C31 119.2 mm to (184.3, 120.3), turned to -90 degrees
- moved R2 116.0 mm to (191.0, 79.7), turned to 90 degrees
- moved R29 115.6 mm to (179.6, 121.3), turned to -90 degrees
- moved C4 112.3 mm to (191.0, 77.0), turned to 90 degrees
- moved U2 110.4 mm to (182.7, 124.2), turned to 180 degrees
- moved R28 109.4 mm to (188.5, 123.0), turned to 180 degrees
- moved C32 106.4 mm to (188.3, 128.6), turned to -90 degrees
- moved C3 105.8 mm to (184.2, 77.1), turned to -90 degrees
- moved Y1 102.2 mm to (187.8, 77.0)
- moved C30 100.7 mm to (177.9, 127.2), turned to 90 degrees
- moved BTN6 100.3 mm to (158.0, 109.8), turned to 90 degrees
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Other:
- board outline added: 51 x 82 mm
- copper layers 2 -> 4

Commit message: update rev.2.2
Parts:
- added C36: 2.2u, Capacitor_SMD:C_0402_1005Metric, F.Cu at (161.2, 118.4)
- added J1: USB-TYPE-C-017, our-parts:USB-TYPE-C-SMD_C9900008089, F.Cu at (123.4, 102.3)
- BTN5, BTN6, C19, C20, C6, C7, C9, R11, R12, R13, R14, R16, R17, R20, R21, R3, R5: moved to B.Cu
- C21: moved to F.Cu
- moved R16 129.1 mm to (198.8, 113.9), turned to -90 degrees
- moved R17 125.9 mm to (196.2, 113.9), turned to -90 degrees
- moved C19 122.9 mm to (197.5, 113.9), turned to 90 degrees
- moved C20 119.6 mm to (194.8, 113.9), turned to 90 degrees
- moved C6 91.5 mm to (182.5, 69.1), turned to 90 degrees
- moved C7 88.9 mm to (180.0, 69.1), turned to 90 degrees
- moved C9 85.4 mm to (176.6, 69.2), turned to 90 degrees
- moved R5 82.5 mm to (173.7, 69.2), turned to 90 degrees
- moved C25 80.2 mm to (150.7, 112.4), turned to 90 degrees
- moved C29 74.9 mm to (161.0, 86.2), turned to -90 degrees
- moved C23 68.1 mm to (139.0, 112.0), turned to 180 degrees
- moved C26 68.0 mm to (150.9, 90.0), turned to 90 degrees
- moved C24 66.2 mm to (139.0, 110.7)
- moved C32 65.1 mm to (123.6, 121.4), turned to 180 degrees
- moved E1 62.3 mm to (195.9, 117.6), turned to 0 degrees
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Other:
- board size 51 x 82 mm -> 82 x 51 mm

Commit message: update rev.2.21
Parts:
- moved C32 2.51 mm to (125.5, 123.1), turned to -90 degrees
- moved L2 0.11 mm to (122.3, 115.9)
- turned R25 to 90 degrees
- turned R26 to 90 degrees
Routing:
- net Net-(U7-PGOOD): track 0.00 -> 16.8 mm, vias 0 -> 1
- net +BATT: track 0.00 -> 16.6 mm
- net VBUS: track 0.00 -> 14.4 mm, vias 0 -> 3
- net Net-(U7-CHG): track 0.00 -> 14.0 mm, vias 0 -> 1
- net +3V3: track 0.00 -> 10.9 mm
- net VCC: track 0.00 -> 8.14 mm, vias 0 -> 1
- net BTN3: track 0.00 -> 6.60 mm
- net BTN4: track 0.00 -> 5.91 mm
- net BTN6: track 0.00 -> 4.81 mm
- net Net-(U2-FB): track 0.00 -> 4.71 mm
- net BTN5: track 0.00 -> 4.45 mm
- net BTN2: track 0.00 -> 4.28 mm
- net BTN1: track 0.00 -> 3.70 mm
- net Net-(J1-CC1): track 0.00 -> 2.63 mm
- net Net-(J1-CC2): track 0.00 -> 2.60 mm
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- added copper zone on B.Cu, net Net-(L2-Pad1)
- added copper zone on B.Cu, net Net-(L2-Pad2)
- added copper zone on B.Cu, net VCC

Commit message: update rev.2.22
Parts:
- moved R15 18.1 mm to (186.1, 104.5), turned to 0 degrees
- moved C17 16.4 mm to (180.5, 94.4), turned to 90 degrees
- moved C18 16.2 mm to (172.7, 94.4), turned to 90 degrees
- moved R7 15.8 mm to (175.3, 109.3), turned to 90 degrees
- moved R8 15.6 mm to (176.3, 109.3), turned to 90 degrees
- moved C16 15.3 mm to (179.2, 94.4), turned to 90 degrees
- moved C12 15.1 mm to (174.0, 94.4), turned to 90 degrees
- moved C15 14.5 mm to (177.9, 94.4), turned to 90 degrees
- moved C13 14.5 mm to (175.3, 94.4), turned to 90 degrees
- moved C14 14.3 mm to (176.6, 94.4), turned to 90 degrees
- moved C11 13.9 mm to (170.0, 98.7), turned to 180 degrees
- moved C10 13.3 mm to (170.0, 99.8), turned to 180 degrees
- moved C8 13.1 mm to (170.0, 100.8), turned to 180 degrees
- moved L1 11.8 mm to (178.2, 107.2), turned to 0 degrees
- moved U1 1.16 mm to (176.5, 101.0), turned to 0 degrees
Routing:
- net LCD_LED: track 0.00 -> 17.4 mm, vias 0 -> 2
- net LCD_SCK: track 0.00 -> 14.8 mm
- net LCD_SDA: track 0.00 -> 14.0 mm
- net LCD_A0: track 0.00 -> 13.4 mm
- net LCD_RESET: track 0.00 -> 12.5 mm
- net +3V3: track 10.9 -> 22.4 mm
- net +1V1: track 0.00 -> 5.94 mm, vias 0 -> 1
- net PUPPY_WIFI_EN: track 0.00 -> 4.86 mm
- net Net-(D1-A): track 0.00 -> 1.60 mm
- added copper zone on B.Cu, net +3V3

Commit message: update rev.2.3
Parts:
- moved C32 2.32 mm to (125.8, 120.8), turned to 180 degrees
- moved R27 1.88 mm to (128.8, 122.5), turned to -90 degrees
- moved R7 1.58 mm to (173.7, 109.4)
- moved R8 1.48 mm to (174.8, 109.4)
- moved R28 1.00 mm to (130.1, 122.1)
- moved R30 0.70 mm to (130.6, 120.0)
- moved C31 0.62 mm to (131.3, 117.3)
- moved L1 0.27 mm to (178.2, 107.0)
Connections:
- U7 pad 2: +BATT -> (no net)
Routing:
- net /USB_D-: track 0.00 -> 75.2 mm, vias 0 -> 2
- net /USB_D+: track 0.00 -> 70.1 mm, vias 0 -> 2
- net VCC: track 8.14 -> 47.4 mm, vias 1 -> 6
- net LCD_PUPPY_SELECT: track 0.00 -> 32.8 mm
- net PUPPY_WIFI_BOOT: track 0.00 -> 17.7 mm
- net GND: track 0.00 -> 17.6 mm, vias 0 -> 14
- net VBUS: track 14.4 -> 21.7 mm, vias 3 -> 9
- net +3V3: track 22.4 -> 17.1 mm, vias 0 -> 10
- net (no net): track 0.00 -> 4.98 mm
- net ENC-A: track 0.00 -> 4.85 mm
- net ENC-B: track 0.00 -> 4.68 mm
- net +BATT: track 16.6 -> 19.1 mm
- net Net-(U7-ILIM): track 0.00 -> 1.40 mm
- net Net-(R31-Pad2): track 0.00 -> 1.18 mm
- net Net-(U2-VinA): track 1.94 -> 1.31 mm
- added copper zone on B.Cu, net +BATT
- added copper zone on F.Cu, net /USB_D+
- added copper zone on B.Cu, net ENC-A
- added copper zone on B.Cu, net ENC-B
- added copper zone on B.Cu, net GND
- added copper zone on B.Cu, net VBUS
- added copper zone on F.Cu, net VBUS
- added copper zone on In1.Cu, net VBUS
- added copper zone on F.Cu, net VCC

Commit message: update rev.2.4
Parts:
- added J6: audio-out, our-parts:2.54mm-2PIN, F.Cu at (163.6, 101.1)
- C10, C12, C13, C14, C15, C18: moved to B.Cu
- R15, R20, R21: moved to F.Cu
- moved R16 90.6 mm to (119.8, 69.6), turned to 90 degrees
- moved E1 89.5 mm to (122.7, 66.0), turned to 180 degrees
- moved C32 88.7 mm to (192.9, 62.7), turned to 0 degrees
- moved L2 88.4 mm to (196.4, 67.6), turned to 90 degrees
- moved C19 88.3 mm to (121.1, 69.6), turned to -90 degrees
- moved R27 86.7 mm to (189.9, 61.0), turned to 90 degrees
- moved R17 86.1 mm to (122.4, 69.6), turned to 90 degrees
- moved R28 84.3 mm to (188.6, 61.4), turned to -90 degrees
- moved C20 83.7 mm to (123.8, 69.6), turned to -90 degrees
- moved C35 81.5 mm to (120.9, 78.2), turned to 90 degrees
- moved R30 80.5 mm to (188.1, 63.6), turned to 180 degrees
- moved U2 79.0 mm to (190.6, 67.7), turned to -90 degrees
- moved J3 78.9 mm to (196.8, 104.0), turned to 90 degrees
- moved C30 78.7 mm to (193.7, 72.5), turned to 180 degrees
- moved C34 77.2 mm to (123.0, 78.7), turned to 90 degrees
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Connections:
- U7 pad 11: (no net) -> VCC
- U7 pad 2: (no net) -> +BATT
- U7 pad 3: (no net) -> +BATT
- U7 pad 8: (no net) -> GND
Routing:
- net +BATT: track 19.1 -> 89.1 mm, vias 0 -> 2
- net GND: track 17.6 -> 70.9 mm, vias 14 -> 42
- net BTN_START: track 0.00 -> 47.3 mm, vias 0 -> 3
- net +3V3: track 17.1 -> 63.0 mm, vias 10 -> 29
- net /QSPI_SD2: track 0.00 -> 40.9 mm
- net /QSPI_SD0: track 0.00 -> 40.9 mm, vias 0 -> 4
- net /QSPI_SCLK: track 0.00 -> 38.5 mm, vias 0 -> 4
- net PUPPY_WIFI_EN: track 4.86 -> 42.4 mm, vias 0 -> 2
- net /QSPI_SD1: track 0.00 -> 37.1 mm
- net /GPIO10: track 0.00 -> 36.0 mm
- net /GPIO11: track 0.00 -> 36.0 mm, vias 0 -> 1
- net /GPIO9: track 0.00 -> 30.9 mm, vias 0 -> 1
- net Audio: track 0.00 -> 30.0 mm
- net PUPPY_TX: track 0.00 -> 29.6 mm
- net /GPIO8: track 0.00 -> 29.4 mm
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- added copper zone on B.Cu, net +1V1
- added copper zone on B.Cu, net /VREG_LX
- added copper zone on In2.Cu, net GND
Other:
- board text added: "3V3"
- board text added: "Bypas BAT"
- board text added: "GND"
- board text added: "VCC"

Commit message: update rev.2.5
Parts:
- moved C12 3.34 mm to (136.8, 86.0), turned to 180 degrees
- moved C13 3.12 mm to (136.8, 87.1), turned to 180 degrees
- moved R6 0.06 mm to (122.3, 98.2)
Routing:
- net BTN2: track 4.28 -> 99.8 mm, vias 0 -> 3
- net BTN4: track 5.91 -> 99.7 mm, vias 0 -> 1
- net BTN1: track 3.70 -> 74.8 mm, vias 0 -> 3
- net BTN3: track 6.60 -> 74.3 mm, vias 0 -> 3
- net /GPIO29_ADC3: track 6.93 -> 67.6 mm
- net /GPIO27_ADC1: track 5.29 -> 65.5 mm
- net /GPIO28_ADC2: track 6.17 -> 65.6 mm
- net GND: track 70.9 -> 122.5 mm, vias 42 -> 56
- net BTN5: track 4.45 -> 55.8 mm, vias 0 -> 2
- net /QSPI_SS: track 14.4 -> 58.2 mm, vias 0 -> 2
- net BTN_ESC: track 0.00 -> 42.4 mm, vias 0 -> 3
- net BTN6: track 4.81 -> 42.7 mm, vias 0 -> 3
- net ENC-A: track 4.85 -> 41.4 mm, vias 0 -> 1
- net +1V1: track 18.9 -> 50.6 mm
- net ENC-B: track 4.68 -> 33.2 mm
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- added copper zone on In1.Cu, net +3V3
Other:
- board text added: "Audio"
- board text added: "BOOT"
- board text added: "ESC"
- board text added: "RUN"
- board text added: "START"
