File: VGC-0_rp_1v0/VGC-0_rp_1v0.kicad_pcb (KiCad board)
At the start: 4 copper layers, 82 x 51 mm, 102 parts, among them J1 USB-TYPE-C-017, J2 THT pins for BATTERY, J3 SMD pads for 3.3V, J4 SM03B-SRSS-TB, J6 audio-out, SW1 SW_Push, SW2 SW_Push, SW3 SW_Push, SW4 SW_Push, U1 RP2350_60QFN, U2 RT6154A, U3 W25Q128JVS, U4 ESP8684-MINI-1, U5 APS1604M-3SQR-ZR, U7 BQ24073RGTR, Y1 ABM8-272-T3

Commit message: update rev.2.51
Routing:
- net BTN4: track 99.7 -> 98.1 mm
Changed lines of the file:
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@@
 	)
 	(segment
-		(start 162.917456 68.317456)
-		(end 171.792544 77.192544)
+		(start 169.7 75.35)
+		(end 169.7 82.432811)
+		(width 0.2)
+		(layer "B.Cu")
+		(net 12)
+	)
+	(segment
+		(start 169.7 82.432811)
+		(end 175.642544 88.375355)
 		(width 0.2)
 		(layer "B.Cu")
@@
 	)
 	(segment
-		(start 162.152544 68.317456)
-		(end 162.917456 68.317456)
-		(width 0.2)
-		(layer "B.Cu")
-		(net 12)
-	)
-	(segment
 		(start 137.476304 84.570002)
 		(end 137.131306 84.915)
@@
 	)
 	(segment
-		(start 171.792544 77.192544)
-		(end 171.792544 84.525355)
+		(start 162.152544 68.317456)
+		(end 162.667456 68.317456)
 		(width 0.2)
 		(layer "B.Cu")
@@
 	)
 	(segment
-		(start 171.792544 84.525355)
-		(end 175.642544 88.375355)
+		(start 162.667456 68.317456)
+		(end 169.7 75.35)
 		(width 0.2)
 		(layer "B.Cu")
@@
 	)
 	(segment
-		(start 171.45 90.45)
+		(start 180.122544 74.105355)
+		(end 183.392544 77.375355)
+		(width 0.3)
+		(layer "F.Cu")
+		(net 18)
+	)
+	(segment
+		(start 165.55 92.35)
+		(end 166.6 91.3)
+		(width 0.15)
+		(layer "F.Cu")
+		(net 18)
+	)
+	(segment
+		(start 134.85 84.3)
+		(end 136.65 86.1)
+		(width 0.15)
+		(layer "F.Cu")
+		(net 18)
+	)
+	(segment
+		(start 170.6 91.3)
 		(end 183.392544 78.507456)
 		(width 0.15)
@@
 	)
 	(segment
-		(start 144.075736 89.6)
-		(end 151.692463 89.6)
-		(width 0.15)
-		(layer "F.Cu")
-		(net 18)
-	)
-	(segment
-		(start 169.60071 90.45)
-		(end 171.45 90.45)
-		(width 0.15)
-		(layer "F.Cu")
-		(net 18)
-	)
-	(segment
-		(start 141.725 90.525)
-		(end 142.887868 91.687868)
+		(start 155.35 92.35)
+		(end 165.55 92.35)
+		(width 0.15)
+		(layer "F.Cu")
+		(net 18)
+	)
+	(segment
+		(start 166.6 91.3)
+		(end 170.6 91.3)
+		(width 0.15)
+		(layer "F.Cu")
+		(net 18)
+	)
+	(segment
+		(start 136.65 86.1)
+		(end 136.65 90.15)
+		(width 0.15)
+		(layer "F.Cu")
+		(net 18)
+	)
+	(segment
+		(start 140.675 90.525)
+		(end 141.6 89.6)
+		(width 0.15)
+		(layer "F.Cu")
+		(net 18)
+	)
+	(segment
+		(start 180.122544 72.817456)
+		(end 180.122544 74.105355)
+		(width 0.3)
+		(layer "F.Cu")
+		(net 18)
+	)
+	(segment
+		(start 152.6 89.6)
+		(end 155.35 92.35)
+		(width 0.15)
+		(layer "F.Cu")
+		(net 18)
+	)
+	(segment
+		(start 137.025 90.525)
+		(end 140.675 90.525)
+		(width 0.15)
+		(layer "F.Cu")
+		(net 18)
+	)
+	(segment
+		(start 183.392544 78.507456)
+		(end 183.392544 77.375355)
 		(width 0.15)
 		(layer "F.Cu")
@@
 	)
 	(segment
-		(start 180.122544 74.105355)
-		(end 183.392544 77.375355)
-		(width 0.3)
-		(layer "F.Cu")
-		(net 18)
-	)
-	(segment
-		(start 154.542463 92.45)
-		(end 167.60071 92.45)
-		(width 0.15)
-		(layer "F.Cu")
-		(net 18)
-	)
-	(segment
-		(start 137.025 90.525)
-		(end 141.725 90.525)
-		(width 0.15)
-		(layer "F.Cu")
-		(net 18)
-	)
-	(segment
-		(start 143.3 90.375736)
-		(end 144.075736 89.6)
-		(width 0.15)
-		(layer "F.Cu")
-		(net 18)
-	)
-	(segment
-		(start 183.392544 78.507456)
-		(end 183.392544 77.375355)
-		(width 0.15)
-		(layer "F.Cu")
-		(net 18)
-	)
-	(segment
-		(start 180.122544 72.817456)
-		(end 180.122544 74.105355)
-		(width 0.3)
-		(layer "F.Cu")
-		(net 18)
-	)
-	(segment
-		(start 134.85 84.3)
-		(end 136.65 86.1)
-		(width 0.15)
-		(layer "F.Cu")
-		(net 18)
-	)
-	(segment
-		(start 151.692463 89.6)
-		(end 154.542463 92.45)
-		(width 0.15)
-		(layer "F.Cu")
-		(net 18)
-	)
-	(segment
-		(start 167.60071 92.45)
-		(end 169.60071 90.45)
-		(width 0.15)
-		(layer "F.Cu")
-		(net 18)
-	)
-	(segment
-		(start 136.65 86.1)
-		(end 136.65 90.15)
-		(width 0.15)
-		(layer "F.Cu")
-		(net 18)
-	)
-	(segment
-		(start 142.887868 91.687868)
-		(end 143.3 91.275736)
-		(width 0.15)
-		(layer "F.Cu")
-		(net 18)
-	)
-	(segment
-		(start 143.3 91.275736)
-		(end 143.3 90.375736)
+		(start 141.6 89.6)
+		(end 152.6 89.6)
 		(width 0.15)
 		(layer "F.Cu")
@@
 		(drill 0.35)
 		(layers "F.Cu" "B.Cu")
-		(net 18)
-	)
-	(segment
-		(start 177.38323 71.366041)
-		(end 183.392544 77.375355)
-		(width 0.2)
-		(layer "B.Cu")
-		(net 18)
-	)
-	(segment
-		(start 170.866041 71.366041)
-		(end 177.38323 71.366041)
-		(width 0.2)
-		(layer "B.Cu")
 		(net 18)
 	)
@@
 	)
 	(segment
+		(start 171.55 72.05)
+		(end 178.067189 72.05)
+		(width 0.2)
+		(layer "B.Cu")
+		(net 18)
+	)
+	(segment
 		(start 134.85 84.3)
 		(end 135.05 84.1)
@@
 	)
 	(segment
+		(start 164.917456 65.417456)
+		(end 171.55 72.05)
+		(width 0.2)
+		(layer "B.Cu")
+		(net 18)
+	)
+	(segment
+		(start 162.152544 65.417456)
+		(end 164.917456 65.417456)
+		(width 0.2)
+		(layer "B.Cu")
+		(net 18)
+	)
+	(segment
 		(start 137.048889 84.148889)
 		(end 137.427776 83.770002)
@@
 	)
 	(segment
-		(start 162.152544 65.417456)
-		(end 164.917456 65.417456)
-		(width 0.2)
-		(layer "B.Cu")
-		(net 18)
-	)
-	(segment
 		(start 135.05 84.1)
 		(end 136.565074 84.1)
@@
 	)
 	(segment
+		(start 178.067189 72.05)
+		(end 183.392544 77.375355)
+		(width 0.2)
+		(layer "B.Cu")
+		(net 18)
+	)
+	(segment
 		(start 137.427776 83.770002)
 		(end 138.712351 83.770002)
 		(width 0.15)
-		(layer "B.Cu")
-		(net 18)
-	)
-	(segment
-		(start 164.917456 65.417456)
-		(end 170.866041 71.366041)
-		(width 0.2)
 		(layer "B.Cu")
 		(net 18)
@@
 	)
 	(segment
-		(start 125.385 95.602897)
+		(start 125.75 95.237897)
 		(end 122.81 98.177897)
 		(width 0.15)
@@
 	(segment
 		(start 128.65 77.1)
-		(end 125.385 80.365)
+		(end 125.75 80)
 		(width 0.15)
 		(layer "F.Cu")
@@
 	)
 	(segment
-		(start 125.385 80.365)
-		(end 125.385 95.602897)
-		(width 0.15)
-		(layer "F.Cu")
+		(start 125.75 80)
+		(end 125.75 95.237897)
+		(width 0.15)
+		(layer "F.Cu")
